File: kicad/Desk Buddy.kicad_sch (KiCad schematic)
At the start: 0 parts

Commit message: Create hierarchical sheet skeleton (9 sheets)
Root sheet holds 9 empty subsheets matching schematic-notes.md's
subsystem breakdown (Power, MCU, Display, two sensor buses, LED,
Audio, Motor, misc I/O). No hierarchical sheet pins used -- cross-
sheet nets will be wired with global labels per the KiCad plan.

Also ignore .history/ (a local-history editor artifact that showed
up as a nested git repo, unrelated to the project).

Co-Authored-By: Claude Sonnet 5 <noreply@anthropic.com>
Other:
- added sheet 00_Power (00_Power.kicad_sch)
- added sheet 01_MCU (01_MCU.kicad_sch)
- added sheet 02_Display (02_Display.kicad_sch)
- added sheet 03_Sensors_I2C0 (03_Sensors_I2C0.kicad_sch)
- added sheet 04_Sensors_I2C1_Expansion (04_Sensors_I2C1_Expansion.kicad_sch)
- added sheet 05_LED (05_LED.kicad_sch)
- added sheet 06_Audio (06_Audio.kicad_sch)
- added sheet 07_Motor (07_Motor.kicad_sch)
- added sheet 08_Misc_IO (08_Misc_IO.kicad_sch)
