File: kicad/06_Audio.kicad_sch (KiCad schematic)
At the start: 0 parts

Commit message: Wire 06_Audio: MAX98357A + 6-pin JST
VCC to VBAT_OUT, GND, and BCLK/LRC/DIN/SD to their matching I2S_*
global labels. GAIN left unrouted (NC on the module itself, 15dB
default).

ERC: 0 errors, 6 warnings, all isolated labels for sheets not yet
wired -- 4 fewer than before (all four I2S_* labels resolved).

Co-Authored-By: Claude Sonnet 5 <noreply@anthropic.com>
Parts:
- added J12: Conn_01x06, Connector_JST:JST_PH_B6B-PH-K_1x06_P2.00mm_Vertical, symbol Connector_Generic:Conn_01x06
- added U8: (no value), symbol DeskBuddy:MAX98357A
Connections:
- new net GND: J12.2 (Pin_2), U8.2 (GND)
- new net I2S_BCLK: J12.3 (Pin_3), U8.3 (BCLK)
- new net I2S_DIN: J12.5 (Pin_5), U8.5 (DIN)
- new net I2S_LRC: J12.4 (Pin_4), U8.4 (LRC)
- new net I2S_SD: J12.6 (Pin_6), U8.6 (SD)
- new net VBAT_OUT: J12.1 (Pin_1), U8.1 (VCC)
