File: kicad/03_Sensors_I2C0.kicad_sch (KiCad schematic)
At the start: 0 parts

Commit message: Wire 03_Sensors_I2C0: ToF, AHT20+BMP280, MPU6050
Three internal-bus sensors each wired symbol-to-JST on shared nets
(6-pin for ToF incl. INT/SHUT, 4-pin each for AHT20+BMP280 and
MPU6050), all on I2C0_SDA/I2C0_SCL with one pair of 4.7k pull-ups
to 3V3 for the whole bus.

ERC: 0 errors, 14 warnings, all isolated labels for sheets not yet
wired -- 4 fewer than before (I2C0_SDA, I2C0_SCL, TOF_INT, TOF_SHUT
now resolved against 01_MCU).

Co-Authored-By: Claude Sonnet 5 <noreply@anthropic.com>
Parts:
- added J6: ToF, Connector_JST:JST_PH_B6B-PH-K_1x06_P2.00mm_Vertical, symbol Connector_Generic:Conn_01x06
- added J7: AHT+BMP, Connector_JST:JST_PH_B4B-PH-K_1x04_P2.00mm_Vertical, symbol Connector_Generic:Conn_01x04
- added J8: MPU6050, symbol Connector_Generic:Conn_01x04
- added R15, R16: 4.7k, Resistor_THT:R_Array_SIP4, symbol Device:R_Small
- added U6: (no value), symbol DeskBuddy:TOF050C
- added U7: (no value), symbol DeskBuddy:AHT20+BMP280
Connections:
- new net +3V3: J6.1 (Pin_1), J7.1 (Pin_1), J8.1 (Pin_1), R15.1, R16.1, U6.1 (VIN), U7.1 (VDD)
- new net GND: J6.2 (Pin_2), J7.3 (Pin_3), J8.2 (Pin_2), U6.2 (GND), U7.3 (GND)
- new net I2C0_SCL: J6.4 (Pin_4), J7.4 (Pin_4), J8.4 (Pin_4), R16.2, U6.4 (SCL), U7.4 (SCL)
- new net I2C0_SDA: J6.3 (Pin_3), J7.2 (Pin_2), J8.3 (Pin_3), R15.2, U6.3 (SDA), U7.2 (SDA)
- new net TOF_INT: J6.5 (Pin_5), U6.5 (INT)
- new net TOF_SHUT: J6.6 (Pin_6), U6.6 (SHUT)

Commit message: Footprint atamaları düzeltildi, satın alım listesi eklendi
- R/C/LED 0805, USB-C USB4110, tactile switch PTS645SM43SMTR92
- C6 47uF 1206, D5 BAT54 yerine SS14 (SMA)
- J8 JST ve TestPoint footprint'leri atandı
- purchase-list.md eklendi, BOM/plan/notlar güncellendi

Co-Authored-By: Claude Sonnet 5.5 <noreply@anthropic.com>
Parts:
- J8: footprint (none) -> Connector_JST:JST_PH_B4B-PH-K_1x04_P2.00mm_Vertical
- R15, R16: footprint Resistor_THT:R_Array_SIP4 -> Resistor_SMD:R_0805_2012Metric
Changed lines of the file:
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@@
 			)
 		)
-		(property "Footprint" "Resistor_THT:R_Array_SIP4"
+		(property "Footprint" "Resistor_SMD:R_0805_2012Metric"
 			(at 165.1 41.91 0)
 			(hide yes)
@@
 			)
 		)
-		(property "Footprint" "Resistor_THT:R_Array_SIP4"
+		(property "Footprint" "Resistor_SMD:R_0805_2012Metric"
 			(at 165.1 45.72 0)
 			(hide yes)
@@
 			)
 		)
-		(property "Footprint" ""
+		(property "Footprint" "Connector_JST:JST_PH_B4B-PH-K_1x04_P2.00mm_Vertical"
 			(at 120.65 57.15 0)
 			(hide yes)
