File: kicad/04_Sensors_I2C1_Expansion.kicad_sch (KiCad schematic)
At the start: 0 parts

Commit message: Wire 04_Sensors_I2C1_Expansion: two parallel external JST ports
Both 4-pin JSTs wired identically (VCC/GND/SDA/SCL) onto the same
isolated I2C1 bus, with one pair of 4.7k pull-ups to 3V3. No
sensors on this sheet by design -- it's the open expansion port for
future I2C devices or the planned mini-gamepads.

ERC: 0 errors, 12 warnings, all isolated labels for sheets not yet
wired -- 2 fewer than before (I2C1_SDA, I2C1_SCL now resolved).

Co-Authored-By: Claude Sonnet 5 <noreply@anthropic.com>
Parts:
- added J10: EXP_I2C1_2, Connector_JST:JST_PH_B4B-PH-K_1x04_P2.00mm_Vertical, symbol Connector_Generic:Conn_01x04
- added J9: EXP_I2C1_1, Connector_JST:JST_PH_B4B-PH-K_1x04_P2.00mm_Vertical, symbol Connector_Generic:Conn_01x04
- added R17, R18: 4.7k, Resistor_THT:R_Array_SIP4, symbol Device:R_Small
Connections:
- new net +3V3: J10.1 (Pin_1), J9.1 (Pin_1), R17.2, R18.2
- new net GND: J10.2 (Pin_2), J9.2 (Pin_2)
- new net I2C1_SCL: J10.4 (Pin_4), J9.4 (Pin_4), R18.1
- new net I2C1_SDA: J10.3 (Pin_3), J9.3 (Pin_3), R17.1

Commit message: Footprint atamaları düzeltildi, satın alım listesi eklendi
- R/C/LED 0805, USB-C USB4110, tactile switch PTS645SM43SMTR92
- C6 47uF 1206, D5 BAT54 yerine SS14 (SMA)
- J8 JST ve TestPoint footprint'leri atandı
- purchase-list.md eklendi, BOM/plan/notlar güncellendi

Co-Authored-By: Claude Sonnet 5.5 <noreply@anthropic.com>
Parts:
- R17, R18: footprint Resistor_THT:R_Array_SIP4 -> Resistor_SMD:R_0805_2012Metric
Changed lines of the file:
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@@
 			)
 		)
-		(property "Footprint" "Resistor_THT:R_Array_SIP4"
+		(property "Footprint" "Resistor_SMD:R_0805_2012Metric"
 			(at 106.68 43.18 0)
 			(hide yes)
@@
 			)
 		)
-		(property "Footprint" "Resistor_THT:R_Array_SIP4"
+		(property "Footprint" "Resistor_SMD:R_0805_2012Metric"
 			(at 106.68 36.83 0)
 			(hide yes)
