File: kicad/05_LED.kicad_sch (KiCad schematic)
At the start: 0 parts

Commit message: Wire 05_LED: onboard WS2812B chain + external JST output
Two onboard WS2812B daisy-chained (DIN from WS2812_ONBOARD, DOUT1->
DIN2, DOUT2 no-connect at end of chain), both powered from VBAT_OUT.
External 3-pin JST carries VBAT_OUT/GND/data, with a 330R series
resistor between WS2812_EXT and the JST's data pin for signal
integrity on the longer external run.

ERC: 0 errors, 10 warnings, all isolated labels for sheets not yet
wired -- 2 fewer than before (WS2812_ONBOARD, WS2812_EXT resolved).

Co-Authored-By: Claude Sonnet 5 <noreply@anthropic.com>
Parts:
- added D1, D4: WS2812B, LED_SMD:LED_WS2812B_PLCC4_5.0x5.0mm_P3.2mm, symbol LED:WS2812B
- added J11: EXT_LED, Connector_JST:JST_PH_B3B-PH-K_1x03_P2.00mm_Vertical, symbol Connector_Generic:Conn_01x03
- added R19: 330, Resistor_THT:R_Array_SIP4, symbol Device:R_Small
Connections:
- new net: D1.2 (DOUT), D4.4 (DIN)
- new net: J11.3 (Pin_3), R19.2
- new net GND: D1.3 (VSS), D4.3 (VSS), J11.2 (Pin_2)
- new net VBAT_OUT: D1.1 (VDD), D4.1 (VDD), J11.1 (Pin_1)
- new net WS2812_EXT: R19.1
- new net WS2812_ONBOARD: D1.4 (DIN)
- no-connect marks 0 -> 1

Commit message: Footprint atamaları düzeltildi, satın alım listesi eklendi
- R/C/LED 0805, USB-C USB4110, tactile switch PTS645SM43SMTR92
- C6 47uF 1206, D5 BAT54 yerine SS14 (SMA)
- J8 JST ve TestPoint footprint'leri atandı
- purchase-list.md eklendi, BOM/plan/notlar güncellendi

Co-Authored-By: Claude Sonnet 5.5 <noreply@anthropic.com>
Parts:
- R19: footprint Resistor_THT:R_Array_SIP4 -> Resistor_SMD:R_0805_2012Metric
Changed lines of the file:
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@@
 			)
 		)
-		(property "Footprint" "Resistor_THT:R_Array_SIP4"
+		(property "Footprint" "Resistor_SMD:R_0805_2012Metric"
 			(at 58.42 80.01 0)
 			(hide yes)
