File: kicad/07_Motor.kicad_sch (KiCad schematic)
At the start: 0 parts

Commit message: Wire 07_Motor: vibration motor switch with flyback protection
AO3400A low-side switch (gate via 100R from MOTOR_PWM, 10k pull-down
to default off at boot), BAT54 Schottky across the motor terminals
(cathode to VBAT_OUT, anode to the switched node) to clamp turn-off
inductive kickback, 2-pin JST to the motor.

ERC: 0 errors, 5 warnings -- MOTOR_PWM now resolved, leaving exactly
the 5 labels that belong to the last sheet, 08_Misc_IO.

Co-Authored-By: Claude Sonnet 5 <noreply@anthropic.com>
Parts:
- added D5: BAT54, Package_TO_SOT_SMD:SOT-23, symbol Device:D_Schottky
- added J13: Motor, Connector_JST:JST_PH_B2B-PH-K_1x02_P2.00mm_Vertical, symbol Connector_Generic:Conn_01x02
- added Q2: AO3400A, Package_TO_SOT_SMD:SOT-23, symbol Transistor_FET:AO3400A
- added R20: 100, Resistor_THT:R_Array_SIP4, symbol Device:R_Small
- added R21: 10k, Resistor_THT:R_Array_SIP4, symbol Device:R_Small
Connections:
- new net: D5.2 (A), J13.2 (Pin_2), Q2.3 (D)
- new net: Q2.1 (G), R20.2, R21.2
- new net GND: Q2.2 (S), R21.1
- new net MOTOR_PWM: R20.1
- new net VBAT_OUT: D5.1 (K), J13.1 (Pin_1)

Commit message: Footprint atamaları düzeltildi, satın alım listesi eklendi
- R/C/LED 0805, USB-C USB4110, tactile switch PTS645SM43SMTR92
- C6 47uF 1206, D5 BAT54 yerine SS14 (SMA)
- J8 JST ve TestPoint footprint'leri atandı
- purchase-list.md eklendi, BOM/plan/notlar güncellendi

Co-Authored-By: Claude Sonnet 5.5 <noreply@anthropic.com>
Parts:
- D5: value BAT54 -> SS14; footprint Package_TO_SOT_SMD:SOT-23 -> Diode_SMD:D_SMA
- R20, R21: footprint Resistor_THT:R_Array_SIP4 -> Resistor_SMD:R_0805_2012Metric
Changed lines of the file:
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@@
 			)
 		)
-		(property "Footprint" "Resistor_THT:R_Array_SIP4"
+		(property "Footprint" "Resistor_SMD:R_0805_2012Metric"
 			(at 57.15 60.96 0)
 			(hide yes)
@@
 			)
 		)
-		(property "Value" "BAT54"
+		(property "Value" "SS14"
 			(at 92.71 47.9424 90)
 			(show_name no)
@@
 			)
 		)
-		(property "Footprint" "Package_TO_SOT_SMD:SOT-23"
+		(property "Footprint" "Diode_SMD:D_SMA"
 			(at 90.17 46.99 0)
 			(hide yes)
@@
 			)
 		)
-		(property "Footprint" "Resistor_THT:R_Array_SIP4"
+		(property "Footprint" "Resistor_SMD:R_0805_2012Metric"
 			(at 57.15 66.04 0)
 			(hide yes)
