File: kicad/08_Misc_IO.kicad_sch (KiCad schematic)
At the start: 0 parts

Commit message: Wire 08_Misc_IO: complete the schematic -- full project ERC clean
LDR (off-board, 2-pin JST + onboard 10k divider tapped by LDR_ADC),
two TTP223 touch sensors (3-pin JST each, OUT to TTP223_1/2), and a
4-pin UART breakout (3V3/GND/TX/RX). This was the last unwired
sheet.

Full project ERC: 0 errors, 0 warnings across all 9 sheets. Every
peripheral from BOM.md is captured and connected per the locked
GPIO map in schematic-notes.md. Schematic capture is done; next up
is PCB layout.

Also updates plan.md's KiCad section to reflect the finished
schematic phase.

Co-Authored-By: Claude Sonnet 5 <noreply@anthropic.com>
Parts:
- added J14: Conn_01x02, Connector_JST:JST_PH_B2B-PH-K_1x02_P2.00mm_Vertical, symbol Connector_Generic:Conn_01x02
- added J15: TTP_1, Connector_JST:JST_PH_B3B-PH-K_1x03_P2.00mm_Vertical, symbol Connector_Generic:Conn_01x03
- added J16: TTP_2, Connector_JST:JST_PH_B3B-PH-K_1x03_P2.00mm_Vertical, symbol Connector_Generic:Conn_01x03
- added J17: UART, Connector_JST:JST_PH_B4B-PH-K_1x04_P2.00mm_Vertical, symbol Connector_Generic:Conn_01x04
- added R22: LDR, symbol Device:R_Photo
- added R23: 10k, Resistor_THT:R_Array_SIP4, symbol Device:R_Small
- added U10, U9: (no value), symbol DeskBuddy:TTP223
Connections:
- new net +3V3: J15.1 (Pin_1), J16.1 (Pin_1), J17.1 (Pin_1), R23.1, U10.1 (VCC), U9.1 (VCC)
- new net GND: J14.2 (Pin_2), J15.2 (Pin_2), J16.2 (Pin_2), J17.2 (Pin_2), R22.2, U10.2 (GND), U9.2 (GND)
- new net LDR_ADC: J14.1 (Pin_1), R22.1, R23.2
- new net TTP223_1: J15.3 (Pin_3), U9.3 (OUT)
- new net TTP223_2: J16.3 (Pin_3), U10.3 (OUT)
- new net UART_RX: J17.4 (Pin_4)
- new net UART_TX: J17.3 (Pin_3)

Commit message: Footprint atamaları düzeltildi, satın alım listesi eklendi
- R/C/LED 0805, USB-C USB4110, tactile switch PTS645SM43SMTR92
- C6 47uF 1206, D5 BAT54 yerine SS14 (SMA)
- J8 JST ve TestPoint footprint'leri atandı
- purchase-list.md eklendi, BOM/plan/notlar güncellendi

Co-Authored-By: Claude Sonnet 5.5 <noreply@anthropic.com>
Parts:
- R23: footprint Resistor_THT:R_Array_SIP4 -> Resistor_SMD:R_0805_2012Metric
Changed lines of the file:
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@@
 			)
 		)
-		(property "Footprint" "Resistor_THT:R_Array_SIP4"
+		(property "Footprint" "Resistor_SMD:R_0805_2012Metric"
 			(at 138.43 27.94 0)
 			(hide yes)
