File: kicad/01_MCU.kicad_sch (KiCad schematic)
At the start: 0 parts

Commit message: Wire 01_MCU: ESP32-S3, boot/reset/power buttons, all GPIO labels
ESP32-S3-WROOM-1 with VDD3P3 bulk cap, three button circuits
(EN/reset with debounce cap, IO0/boot, IO2/power - all 10k pull-up
to 3V3), USB_D-/USB_D+ tied to 00_Power's global labels, and a
global label on every remaining assigned GPIO matching the locked
pin table (LCD_*, I2C0_*, I2C1_*, I2S_*, TOF_*, TTP223_*, UART_*,
WS2812_*, MOTOR_PWM, LDR_ADC, CHG_CE, VBAT_SENSE). IO45/IO46 left
untouched (strapping). Added a 3-pin header (3V3/GND/GPIO48_SPARE)
for the one free GPIO, and two TestPoint pads (3V3, VBAT_OUT) on
00_Power for quick multimeter access.

ERC: 0 errors, 27 warnings -- all "label connected to only one pin"
on the peripheral-facing global labels waiting on their own sheets
(02_Display through 08_Misc_IO), exactly the expected set with no
unexplained entries.

Co-Authored-By: Claude Sonnet 5 <noreply@anthropic.com>
Parts:
- added C6: 47uF, symbol Device:C_Small
- added C7: 100nF, symbol Device:C_Small
- added J3: GPIO48, Connector_PinHeader_2.54mm:PinHeader_1x03_P2.54mm_Vertical, symbol Connector_Generic:Conn_01x03
- added R10, R11, R12: 10k, symbol Device:R_Small
- added SW1: Push_EN, RF_Module:ESP32-S3-WROOM-1, symbol Switch:SW_Push
- added SW2: Push_BOOT, RF_Module:ESP32-S3-WROOM-1, symbol Switch:SW_Push
- added SW3: Switch_POWER, RF_Module:ESP32-S3-WROOM-1, symbol Switch:SW_Push
- added U4: ESP32-S3-WROOM-1, RF_Module:ESP32-S3-WROOM-1, symbol RF_Module:ESP32-S3-WROOM-1
Connections:
- new net +3V3: C6.1, J3.1 (Pin_1), R10.2, R11.2, R12.2, U4.2 (3V3)
- new net CHG_CE: U4.32 (IO39)
- new net ESP32_BOOT: R11.1, SW2.1, U4.27 (IO0)
- new net ESP32_EN: C7.1, R10.1, SW1.1, U4.3 (EN)
- new net ESP32_POWER: R12.1, SW3.1, U4.38 (IO2)
- new net GND: C6.2, C7.2, J3.2 (Pin_2), SW1.2, SW2.2, SW3.2, U4.1 (GND), U4.40 (GND), U4.41 (GND)
- new net GPIO48_SPARE: J3.3 (Pin_3), U4.25 (IO48)
- new net I2C0_SCL: U4.17 (IO9)
- new net I2C0_SDA: U4.12 (IO8)
- new net I2C1_SCL: U4.26 (IO45)
- new net I2C1_SDA: U4.35 (IO42)
- new net I2S_BCLK: U4.8 (IO15)
- new net I2S_DIN: U4.7 (IO7)
- new net I2S_LRC: U4.9 (IO16)
- new net I2S_SD: U4.28 (IO35)
- new net LCD_BL_GATE: U4.4 (IO4)
- new net LCD_CS: U4.18 (IO10)
- new net LCD_DC: U4.22 (IO14)
- new net LCD_MISO: U4.21 (IO13)
- new net LCD_MOSI: U4.19 (IO11)
- new net LCD_RESET: U4.23 (IO21)
- new net LCD_SCK: U4.20 (IO12)
- new net LCD_T_CS: U4.33 (IO40)
- new net LCD_T_IRQ: U4.34 (IO41)
- new net LDR_ADC: U4.39 (IO1)
- new net MOTOR_PWM: U4.29 (IO36)
- new net TOF_INT: U4.11 (IO18)
- new net TOF_SHUT: U4.10 (IO17)
- new net TTP223_1: U4.30 (IO37)
- new net TTP223_2: U4.31 (IO38)
- new net UART_RX: U4.36 (RXD0)
- new net UART_TX: U4.37 (TXD0)
- new net USB_D+: U4.14 (USB_D+)
- new net USB_D-: U4.13 (USB_D-)
- new net VBAT_SENSE: U4.15 (IO3)
- new net WS2812_EXT: U4.6 (IO6)
- new net WS2812_ONBOARD: U4.5 (IO5)
- no-connect marks 0 -> 2

Commit message: Footprint atamaları düzeltildi, satın alım listesi eklendi
- R/C/LED 0805, USB-C USB4110, tactile switch PTS645SM43SMTR92
- C6 47uF 1206, D5 BAT54 yerine SS14 (SMA)
- J8 JST ve TestPoint footprint'leri atandı
- purchase-list.md eklendi, BOM/plan/notlar güncellendi

Co-Authored-By: Claude Sonnet 5.5 <noreply@anthropic.com>
Parts:
- C6: footprint (none) -> Capacitor_SMD:C_1206_3216Metric
- C7: footprint (none) -> Capacitor_SMD:C_0805_2012Metric
- R10, R11, R12: footprint (none) -> Resistor_SMD:R_0805_2012Metric
- SW1, SW2, SW3: footprint RF_Module:ESP32-S3-WROOM-1 -> Button_Switch_SMD:SW_SPST_PTS645Sx43SMTR92
Changed lines of the file:
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@@
 			)
 		)
-		(property "Footprint" ""
+		(property "Footprint" "Resistor_SMD:R_0805_2012Metric"
 			(at 86.36 66.04 0)
 			(hide yes)
@@
 			)
 		)
-		(property "Footprint" "RF_Module:ESP32-S3-WROOM-1"
+		(property "Footprint" "Button_Switch_SMD:SW_SPST_PTS645Sx43SMTR92"
 			(at 88.9 49.53 0)
 			(hide yes)
@@
 			)
 		)
-		(property "Footprint" ""
+		(property "Footprint" "Resistor_SMD:R_0805_2012Metric"
 			(at 88.9 22.86 0)
 			(hide yes)
@@
 			)
 		)
-		(property "Footprint" ""
+		(property "Footprint" "Capacitor_SMD:C_0805_2012Metric"
 			(at 88.9 29.21 0)
 			(hide yes)
@@
 			)
 		)
-		(property "Footprint" "RF_Module:ESP32-S3-WROOM-1"
+		(property "Footprint" "Button_Switch_SMD:SW_SPST_PTS645Sx43SMTR92"
 			(at 88.9 31.75 0)
 			(hide yes)
@@
 			)
 		)
-		(property "Footprint" "RF_Module:ESP32-S3-WROOM-1"
+		(property "Footprint" "Button_Switch_SMD:SW_SPST_PTS645Sx43SMTR92"
 			(at 88.9 67.31 0)
 			(hide yes)
@@
 			)
 		)
-		(property "Footprint" ""
+		(property "Footprint" "Resistor_SMD:R_0805_2012Metric"
 			(at 86.36 48.26 0)
 			(hide yes)
@@
 			)
 		)
-		(property "Footprint" ""
+		(property "Footprint" "Capacitor_SMD:C_1206_3216Metric"
 			(at 171.45 59.69 0)
 			(hide yes)

Commit message: Şematik: I2C1_SCL IO45 yerine IO47'ye bağlandı
I2C1_SCL etiketi strapping pini IO45'e (pin 26) bağlıydı, notlardaki
atama GPIO47 (pin 24). Etiket pin 24'e, no_connect pin 26'ya taşındı.
PCB'de U4 net atamaları güncellendi, şematik parity 0 sorun.

Co-Authored-By: Claude Sonnet 5.5 <noreply@anthropic.com>
Connections:
- net I2C1_SCL: now also U4.24 (IO47); no longer U4.26 (IO45)
Changed lines of the file:
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@@
 	)
 	(no_connect
-		(at 180.34 114.3)
+		(at 180.34 109.22)
 	)
 	(no_connect
@@
 	(global_label "I2C1_SCL"
 		(shape input)
-		(at 180.34 109.22 0)
+		(at 180.34 114.3 0)
 		(fields_autoplaced yes)
 		(effects
@@
 		)
 		(property "Intersheetrefs" "${INTERSHEET_REFS}"
-			(at 192.0942 109.22 0)
+			(at 192.0942 114.3 0)
 			(hide yes)
 			(show_name no)

Commit message: PCB layout Adım 3b: MCU bloğu yerleşimi + harici güç butonu JST'si
- ESP32 anten ucu kart kenarına hizalı, C6/C7/R10, butonlar, pull-up'lar ve J3 yerleştirildi
- Şematik: GPIO2 için 3 pinli JST eklendi (J18 PWR_BTN: 3V3/GND/GPIO2), güç butonunun yanında
- Notlar: yumuşak kapatma güç tüketimi uyarısı, J18 kullanımı
- DRC: bakır/courtyard ihlali yok, şematik parity 0 sorun

Co-Authored-By: Claude Sonnet 5.5 <noreply@anthropic.com>
Parts:
- added J18: PWR_BTN, Connector_JST:JST_PH_B3B-PH-K_1x03_P2.00mm_Vertical, symbol Connector_Generic:Conn_01x03
Connections:
- net +3V3: now also J18.1 (Pin_1)
- net ESP32_POWER: now also J18.3 (Pin_3)
- net GND: now also J18.2 (Pin_2)
Changed lines of the file:
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@@
+		)
+	)
+		(symbol
+		(lib_id "Connector_Generic:Conn_01x03")
+		(at 87.63 111.76 0)
+		(unit 1)
+		(body_style 1)
+		(exclude_from_sim no)
+		(in_bom yes)
+		(on_board yes)
+		(in_pos_files yes)
+		(dnp no)
+		(property "Reference" "J18"
+			(at 89.154 110.49 0)
+			(show_name no)
+			(do_not_autoplace no)
+			(effects
+				(font
+					(size 1.27 1.27)
+				)
+				(justify left)
+			)
+		)
+		(property "Value" "PWR_BTN"
+			(at 89.154 113.03 0)
+			(show_name no)
+			(do_not_autoplace no)
+			(effects
+				(font
+					(size 1.27 1.27)
+				)
+				(justify left)
+			)
+		)
+		(property "Footprint" "Connector_JST:JST_PH_B3B-PH-K_1x03_P2.00mm_Vertical"
+			(at 87.63 111.76 0)
+			(hide yes)
+			(show_name no)
+			(do_not_autoplace no)
+			(effects
+				(font
+					(size 1.27 1.27)
+				)
+			)
+		)
+		(property "Datasheet" ""
+			(at 87.63 111.76 0)
+			(hide yes)
+			(show_name no)
+			(do_not_autoplace no)
+			(effects
+				(font
+					(size 1.27 1.27)
+				)
+			)
+		)
+		(property "Description" "Generic connector, single row, 01x03, script generated (kicad-library-utils/schlib/autogen/connector/)"
+			(at 87.63 111.76 0)
+			(hide yes)
+			(show_name no)
+			(do_not_autoplace no)
+			(effects
+				(font
+					(size 1.27 1.27)
+				)
+			)
+		)
+		(pin "3"
+		)
+		(pin "2"
+		)
+		(pin "1"
+		)
+		(instances
+			(project "Desk Buddy"
+				(path "/4c3424ea-09dd-4711-ada7-066e929b32cd/431db67b-3d56-4cdc-b27f-44a0ba15f32a"
+					(reference "J18")
+					(unit 1)
+				)
+			)
+		)
+	)
+		(symbol
+		(lib_id "power:+3V3")
+		(at 82.55 109.22 90)
+		(unit 1)
+		(body_style 1)
+		(exclude_from_sim no)
+		(in_bom yes)
+		(on_board yes)
+		(in_pos_files yes)
+		(dnp no)
+		(property "Reference" "#PWR060"
+			(at 86.36 109.22 0)
+			(hide yes)
+			(show_name no)
+			(do_not_autoplace no)
+			(effects
+				(font
+					(size 1.27 1.27)
+				)
+			)
+		)
+		(property "Value" "+3V3"
+			(at 80.01 109.22 90)
+			(show_name no)
+			(do_not_autoplace no)
+			(effects
+				(font
+					(size 1.27 1.27)
+				)
+				(justify left)
+			)
+		)
+		(property "Footprint" ""
+			(at 82.55 109.22 0)
+			(hide yes)
+			(show_name no)
+			(do_not_autoplace no)
+			(effects
+				(font
+					(size 1.27 1.27)
+				)
+			)
+		)
+		(property "Datasheet" ""
+			(at 82.55 109.22 0)
+			(hide yes)
+			(show_name no)
+			(do_not_autoplace no)
+			(effects
+				(font
+					(size 1.27 1.27)
+				)
+			)
+		)
+		(property "Description" "Power symbol creates a global label with name \"+3V3\""
+			(at 82.55 109.22 0)
+			(hide yes)
+			(show_name no)
+			(do_not_autoplace no)
+			(effects
+				(font
+					(size 1.27 1.27)
+				)
+			)
+		)
+		(pin "1"
+		)
+		(instances
+			(project "Desk Buddy"
+				(path "/4c3424ea-09dd-4711-ada7-066e929b32cd/431db67b-3d56-4cdc-b27f-44a0ba15f32a"
+					(reference "#PWR060")
+					(unit 1)
+				)
+			)
+		)
+	)
+		(symbol
+		(lib_id "power:GND")
+		(at 82.55 111.76 270)
+		(unit 1)
+		(body_style 1)
+		(exclude_from_sim no)
+		(in_bom yes)
+		(on_board yes)
+		(in_pos_files yes)
+		(dnp no)
+		(property "Reference" "#PWR061"
+			(at 76.2 111.76 0)
+			(hide yes)
+			(show_name no)
+			(do_not_autoplace no)
+			(effects
+				(font
+					(size 1.27 1.27)
+				)
+			)
+		)
+		(property "Value" "GND"
+			(at 77.978 111.76 90)
+			(show_name no)
+			(do_not_autoplace no)
+			(effects
+				(font
+					(size 1.27 1.27)
+				)
+			)
+		)
+		(property "Footprint" ""
+			(at 82.55 111.76 0)
+			(hide yes)
+			(show_name no)
+			(do_not_autoplace no)
+			(effects
+				(font
+					(size 1.27 1.27)
+				)
+			)
+		)
+		(property "Datasheet" ""
+			(at 82.55 111.76 0)
+			(hide yes)
+			(show_name no)
+			(do_not_autoplace no)
+			(effects
+				(font
+					(size 1.27 1.27)
+				)
+			)
+		)
+		(property "Description" "Power symbol creates a global label with name \"GND\" , ground"
+			(at 82.55 111.76 0)
+			(hide yes)
+			(show_name no)
+			(do_not_autoplace no)
+			(effects
+				(font
+					(size 1.27 1.27)
+				)
+			)
+		)
+		(pin "1"
+		)
+		(instances
+			(project "Desk Buddy"
+				(path "/4c3424ea-09dd-4711-ada7-066e929b32cd/431db67b-3d56-4cdc-b27f-44a0ba15f32a"
+					(reference "#PWR061")
+					(unit 1)
+				)
+			)
+		)
+	)
+		(label "ESP32_POWER"
+		(at 82.55 114.3 180)
+		(effects
+			(font
+				(size 1.27 1.27)
+			)
+			(justify right bottom)
 		)
 	)
